Commit message: feat: merge plan_to/execute_to into move_to.py with --plan-only flag

File: srdf/kr_70_r2100.srdf.xacro (robot description, xacro)
@@ -1,4 +1,5 @@
 <?xml version="1.0" ?>
 <robot name="kr_70_r2100" xmlns:xacro="http://www.ros.org/wiki/xacro">
+    <virtual_joint name="virtual_joint" type="fixed" parent_frame="world" child_link="base_link"/>
     <group name="manipulator">
         <joint name="joint_a1"/>

File: urdf/kr_70_r2100.urdf.xacro (robot description, xacro)
@@ -5,4 +5,10 @@
   <xacro:property name="mesh_dir" value="package://kuka_moveit2_spike/meshes"/>
   <!-- ==================== Links ==================== -->
+  <link name="world"/>
+  <joint name="world_to_base" type="fixed">
+    <origin xyz="0 0 0" rpy="0 0 0"/>
+    <parent link="world"/>
+    <child link="base_link"/>
+  </joint>
   <link name="base_link">
     <inertial>

Commit message: Revert "feat: merge plan_to/execute_to into move_to.py with --plan-only flag"
This reverts commit 9a09636ed25600bbb44c74f11dedaf71de4a3d53.

File: srdf/kr_70_r2100.srdf.xacro (robot description, xacro)
@@ -1,5 +1,4 @@
 <?xml version="1.0" ?>
 <robot name="kr_70_r2100" xmlns:xacro="http://www.ros.org/wiki/xacro">
-    <virtual_joint name="virtual_joint" type="fixed" parent_frame="world" child_link="base_link"/>
     <group name="manipulator">
         <joint name="joint_a1"/>

File: urdf/kr_70_r2100.urdf.xacro (robot description, xacro)
@@ -5,10 +5,4 @@
   <xacro:property name="mesh_dir" value="package://kuka_moveit2_spike/meshes"/>
   <!-- ==================== Links ==================== -->
-  <link name="world"/>
-  <joint name="world_to_base" type="fixed">
-    <origin xyz="0 0 0" rpy="0 0 0"/>
-    <parent link="world"/>
-    <child link="base_link"/>
-  </joint>
   <link name="base_link">
     <inertial>
